Commit message: change laser pos

File: definition/sim/hokuyo.urdf.xacro (robot description, xacro)
@@ -5,5 +5,5 @@
     <joint name="laser" type="fixed">
       <axis xyz="0 0 0" />
-      <origin xyz="0.0 0.0 0.43" rpy="0.0 0.0 0.0" />
+      <origin xyz="0.13 0.0 0.21" rpy="0.0 0.0 0.0" />
       <parent link="base_link" />
       <child link="base_laser_link" />

File: definition/sim/kobuki_hexagons_asus_xtion_pro.urdf.xacro (robot description, xacro)
@@ -23,6 +23,6 @@
 <!--  <sensor_hokuyo 		              parent="base_link" name="laser0" ros_topic="scan" update_rate="40" ray_count="1081" min_angle="135" max_angle="-135" />-->
   <include filename="$(find gb_robots)/definition/sim/hokuyo.urdf.xacro" />
-  <xacro:hokuyo name="laser0" parent="base_link" ros_topic="scan" update_rate="40" ray_count="1081" min_angle="135" max_angle="-135">
-      <origin xyz="0.0 0.0 0.08" rpy="${M_PI} 0 0"/>
+  <xacro:hokuyo name="laser0" parent="base_link" ros_topic="scan" update_rate="40" ray_count="1081" min_angle="180" max_angle="-180">
+      <origin xyz="0.13 0.0 0.19" rpy="0 0 0"/>
   </xacro:hokuyo>
 </robot>
